Commit message: update

File: urdf/qbot.xacro (robot description, xacro)
@@ -5,5 +5,5 @@
        xmlns:interface="http://playerstage.sourceforge.net/gazebo/xmlschema/#interface"
        xmlns:xacro="http://ros.org/wiki/xacro"
-	   name="qbot">
+	   name="beagle_bot">
     <property name="M_PI" value="3.14159"/>
     <property name="AX12_LIMIT" value="2.967059729"/>
@@ -103,5 +103,5 @@
 				<origin xyz="${xyz}" rpy="${rpy}" />
 				<geometry>
-					<mesh filename="package://qbot/meshes/ax12_box2.${MESH_EXT}" scale="${M_SCALE} ${M_SCALE} ${M_SCALE}"/>
+					<mesh filename="package://beagle_bot/meshes/ax12_box2.${MESH_EXT}" scale="${M_SCALE} ${M_SCALE} ${M_SCALE}"/>
 				</geometry>
 				<xacro:ax12_color />
@@ -112,5 +112,5 @@
 					<box size="0.032 0.038 0.05" />
 					<!--
-					<mesh filename="package://qbot/meshes/ax12_box2.${MESH_EXT}" scale="${M_SCALE} ${M_SCALE} ${M_SCALE}"/>
+					<mesh filename="package://beagle_bot/meshes/ax12_box2.${MESH_EXT}" scale="${M_SCALE} ${M_SCALE} ${M_SCALE}"/>
 					-->
 				</geometry>
@@ -125,5 +125,5 @@
 				<origin xyz="${xyz}" rpy="${rpy}" />
 				<geometry>
-          			<mesh filename="package://qbot/meshes/F2.${MESH_EXT}" scale="${M_SCALE} ${M_SCALE} ${M_SCALE}"/>
+          			<mesh filename="package://beagle_bot/meshes/F2.${MESH_EXT}" scale="${M_SCALE} ${M_SCALE} ${M_SCALE}"/>
 				</geometry>
 				<xacro:bracket_color />
@@ -134,5 +134,5 @@
 						<box size="0.026 0.05 0.038" />
 						<!--
-          				<mesh filename="package://qbot/meshes/F2.${MESH_EXT}" scale="${M_SCALE} ${M_SCALE} ${M_SCALE}"/>
+          				<mesh filename="package://beagle_bot/meshes/F2.${MESH_EXT}" scale="${M_SCALE} ${M_SCALE} ${M_SCALE}"/>
           				-->
 					</geometry>
@@ -147,5 +147,5 @@
 				<origin xyz="${xyz}" rpy="${rpy}" />
 				<geometry>
-          			<mesh filename="package://qbot/meshes/F3.${MESH_EXT}" scale="${M_SCALE} ${M_SCALE} ${M_SCALE}"/>
+          			<mesh filename="package://beagle_bot/meshes/F3.${MESH_EXT}" scale="${M_SCALE} ${M_SCALE} ${M_SCALE}"/>
 				</geometry>
 				<xacro:bracket_color />
@@ -155,5 +155,5 @@
 					<geometry>
 						<!--
-          				<mesh filename="package://qbot/meshes/F3.${MESH_EXT}" scale="${M_SCALE} ${M_SCALE} ${M_SCALE}"/>
+          				<mesh filename="package://beagle_bot/meshes/F3.${MESH_EXT}" scale="${M_SCALE} ${M_SCALE} ${M_SCALE}"/>
 						-->
 						<box size="0.025 0.04 0.009" />
@@ -386,5 +386,5 @@
     	<origin xyz="0.08 0.05 0.03" rpy="0 0 0" />
 	</joint>
-<gazebo reference="qbot">
+<gazebo reference="beagle_bot">
   	</gazebo>
 </robot>
